Commit message: Finished MotionPlanningGoal. Next, MotionPlanningEnv.

File: tests/pybullet/models/duck.urdf (robot description, URDF)
Before this commit: robot cube.urdf, 1 links, 0 joints
Links:
- link baseLink: geometry collision mesh filename=duck.obj scale=.05 .05 .05; visual mesh filename=duck.obj scale=.05 .05 .05
